File: hardware/display-segment.kicad_sch (KiCad schematic)
At the start: 8 parts, among them Q4 DMP2004VK, U1 P3786E, U2 TLC59284, U3 TLC59284

Commit message: Initial firmware
Parts:
- Q4: footprint Package_TO_SOT_SMD:SOT-563 -> 0-footprints:SOT-563
Changed lines of the file:
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@@
     (pin "9")
     (instances
-      (project "altimeter"
+      (project "navbrick"
         (path "/c26ff3ad-9cdb-4061-8a60-da1ddedb78dd"
           (reference "U3") (unit 1)
@@
     (pin "1")
     (instances
-      (project "altimeter"
+      (project "navbrick"
         (path "/c26ff3ad-9cdb-4061-8a60-da1ddedb78dd/77d6cc85-fb4f-41e1-aad6-e6880a525008/1b9662db-c7fb-4867-bb37-0bbc8541441b"
           (reference "#PWR016") (unit 1)
@@
     (pin "1")
     (instances
-      (project "altimeter"
+      (project "navbrick"
         (path "/c26ff3ad-9cdb-4061-8a60-da1ddedb78dd/77d6cc85-fb4f-41e1-aad6-e6880a525008/1b9662db-c7fb-4867-bb37-0bbc8541441b"
           (reference "#PWR09") (unit 1)
@@
       (effects (font (size 1.27 1.27)) (justify left))
     )
-    (property "Footprint" "Package_TO_SOT_SMD:SOT-563" (at 163.83 41.275 0)
+    (property "Footprint" "0-footprints:SOT-563" (at 163.83 41.275 0)
       (effects (font (size 1.27 1.27) italic) (justify left) hide)
     )
@@
     (pin "5")
     (instances
-      (project "altimeter"
+      (project "navbrick"
         (path "/c26ff3ad-9cdb-4061-8a60-da1ddedb78dd/77d6cc85-fb4f-41e1-aad6-e6880a525008/1b9662db-c7fb-4867-bb37-0bbc8541441b"
           (reference "Q4") (unit 2)
@@
       (effects (font (size 1.27 1.27)) (justify left))
     )
-    (property "Footprint" "Package_TO_SOT_SMD:SOT-563" (at 121.92 41.275 0)
+    (property "Footprint" "0-footprints:SOT-563" (at 121.92 41.275 0)
       (effects (font (size 1.27 1.27) italic) (justify left) hide)
     )
@@
     (pin "5")
     (instances
-      (project "altimeter"
+      (project "navbrick"
         (path "/c26ff3ad-9cdb-4061-8a60-da1ddedb78dd/77d6cc85-fb4f-41e1-aad6-e6880a525008/1b9662db-c7fb-4867-bb37-0bbc8541441b"
           (reference "Q4") (unit 1)
@@
     (pin "2")
     (instances
-      (project "altimeter"
+      (project "navbrick"
         (path "/c26ff3ad-9cdb-4061-8a60-da1ddedb78dd/77d6cc85-fb4f-41e1-aad6-e6880a525008/1b9662db-c7fb-4867-bb37-0bbc8541441b"
           (reference "R9") (unit 1)
@@
     (pin "1")
     (instances
-      (project "altimeter"
+      (project "navbrick"
         (path "/c26ff3ad-9cdb-4061-8a60-da1ddedb78dd/77d6cc85-fb4f-41e1-aad6-e6880a525008/1b9662db-c7fb-4867-bb37-0bbc8541441b"
           (reference "#PWR015") (unit 1)
@@
     (pin "9")
     (instances
-      (project "altimeter"
+      (project "navbrick"
         (path "/c26ff3ad-9cdb-4061-8a60-da1ddedb78dd"
           (reference "U1") (unit 1)
@@
     (pin "1")
     (instances
-      (project "altimeter"
+      (project "navbrick"
         (path "/c26ff3ad-9cdb-4061-8a60-da1ddedb78dd/77d6cc85-fb4f-41e1-aad6-e6880a525008/1b9662db-c7fb-4867-bb37-0bbc8541441b"
           (reference "#PWR012") (unit 1)
@@
     (pin "9")
     (instances
-      (project "altimeter"
+      (project "navbrick"
         (path "/c26ff3ad-9cdb-4061-8a60-da1ddedb78dd"
           (reference "U2") (unit 1)
@@
     (pin "2")
     (instances
-      (project "altimeter"
+      (project "navbrick"
         (path "/c26ff3ad-9cdb-4061-8a60-da1ddedb78dd/77d6cc85-fb4f-41e1-aad6-e6880a525008/1b9662db-c7fb-4867-bb37-0bbc8541441b"
           (reference "R8") (unit 1)
@@
     (pin "1")
     (instances
-      (project "altimeter"
+      (project "navbrick"
         (path "/c26ff3ad-9cdb-4061-8a60-da1ddedb78dd/77d6cc85-fb4f-41e1-aad6-e6880a525008/1b9662db-c7fb-4867-bb37-0bbc8541441b"
           (reference "#PWR010") (unit 1)
@@
     (pin "1")
     (instances
-      (project "altimeter"
+      (project "navbrick"
         (path "/c26ff3ad-9cdb-4061-8a60-da1ddedb78dd/77d6cc85-fb4f-41e1-aad6-e6880a525008/1b9662db-c7fb-4867-bb37-0bbc8541441b"
           (reference "#PWR011") (unit 1)
@@
     (pin "2")
     (instances
-      (project "altimeter"
+      (project "navbrick"
         (path "/c26ff3ad-9cdb-4061-8a60-da1ddedb78dd/77d6cc85-fb4f-41e1-aad6-e6880a525008/1b9662db-c7fb-4867-bb37-0bbc8541441b"
           (reference "C23") (unit 1)
@@
     (pin "1")
     (instances
-      (project "altimeter"
+      (project "navbrick"
         (path "/c26ff3ad-9cdb-4061-8a60-da1ddedb78dd/77d6cc85-fb4f-41e1-aad6-e6880a525008/1b9662db-c7fb-4867-bb37-0bbc8541441b"
           (reference "#PWR013") (unit 1)
@@
     (pin "1")
     (instances
-      (project "altimeter"
+      (project "navbrick"
         (path "/c26ff3ad-9cdb-4061-8a60-da1ddedb78dd/77d6cc85-fb4f-41e1-aad6-e6880a525008/1b9662db-c7fb-4867-bb37-0bbc8541441b"
           (reference "#PWR014") (unit 1)
@@
     (pin "2")
     (instances
-      (project "altimeter"
+      (project "navbrick"
         (path "/c26ff3ad-9cdb-4061-8a60-da1ddedb78dd/77d6cc85-fb4f-41e1-aad6-e6880a525008/1b9662db-c7fb-4867-bb37-0bbc8541441b"
           (reference "C22") (unit 1)
