File: hardware/display-segment.kicad_sch (KiCad schematic)
At the start: 8 parts, among them Q4 DMP2004VK, U1 P3786E, U2 TLC59284, U3 TLC59284

Commit message: Convert to PartDB
Parts:
- C22, C23: symbol 0-passives:C-ceramic -> PartDB:C-Cer-0.1uF-25v-0603; Category (none) -> Capacitors/Ceramic; Manufacturer (none) -> Generic; Part-DB Footprint (none) -> 0603; Part-DB ID (none) -> 4; Part-DB URL (none) -> http://partdb.durbakyta.casa/en/part/4/info; Stock (none) -> 49; Storage Location (none) -> Main Parts Bin; manf (none) -> Generic
- Q4: value DMP2004VK -> DMP2004VK-7; footprint 0-footprints:SOT-563 -> Package_TO_SOT_SMD:SOT-563; symbol 0-semiconductors:DMP2004VK -> PartDB:DMP2004VK-7; Category (none) -> Semiconductors/MOSFETs; DigiKey SPN (none) -> DMP2004VKDICT-ND; MPN (none) -> DMP2004VK-7; Manufacturer (none) -> Diodes Incorporated; Manufacturing Status (none) -> Active; Part-DB ID (none) -> 91; Part-DB URL (none) -> http://partdb.durbakyta.casa/en/part/91/info; Stock (none) -> 7; Storage Location (none) -> Main Parts Bin; digikey# (none) -> DMP2004VKDICT-ND; manf (none) -> Diodes Incorporated; manf# (none) -> DMP2004VK-7
- R8, R9: symbol 0-passives:R -> PartDB:R-2.7k-0.1W-0402; Category (none) -> Resistors; DigiKey SPN (none) -> 10-ERJ-U02F2701XCT-ND; Part-DB Footprint (none) -> 0402; Part-DB ID (none) -> 103; Part-DB URL (none) -> http://partdb.durbakyta.casa/en/part/103/info; Stock (none) -> 0; digikey# (none) -> 10-ERJ-U02F2701XCT-ND
- U15: renamed from U3; value TLC59284 -> TLC59284DBQR; symbol 0-ic-digital:TLC59284 -> PartDB:TLC59284DBQR; Category (none) -> IC/Power; DigiKey SPN (none) -> 296-39245-1-ND; MPN (none) -> TLC59284DBQR; Manufacturer (none) -> Texas Instruments; Manufacturing Status (none) -> Active; Part-DB ID (none) -> 84; Part-DB URL (none) -> http://partdb.durbakyta.casa/en/part/84/info; Stock (none) -> 10; Storage Location (none) -> Main Parts Bin; digikey# (none) -> 296-39245-1-ND; manf (none) -> Texas Instruments; manf# (none) -> TLC59284DBQR
- U16: renamed from U2; value TLC59284 -> TLC59284DBQR; symbol 0-ic-digital:TLC59284 -> PartDB:TLC59284DBQR; Category (none) -> IC/Power; DigiKey SPN (none) -> 296-39245-1-ND; MPN (none) -> TLC59284DBQR; Manufacturer (none) -> Texas Instruments; Manufacturing Status (none) -> Active; Part-DB ID (none) -> 84; Part-DB URL (none) -> http://partdb.durbakyta.casa/en/part/84/info; Stock (none) -> 10; Storage Location (none) -> Main Parts Bin; digikey# (none) -> 296-39245-1-ND; manf (none) -> Texas Instruments; manf# (none) -> TLC59284DBQR
- U53: renamed from U1; value P3786E -> LTP-3786E; footprint 0-footprints:LTP-378x -> am-Displays:LTP-378x; symbol 0-optoelectronics:P3786E -> PartDB:LTP-3786E; Category (none) -> Optoelectronics/LEDs; DigiKey SPN (none) -> 160-1011-ND; MPN (none) -> LTP-3786E; Manufacturer (none) -> Lite-On Inc.; Manufacturing Status (none) -> Active; Part-DB ID (none) -> 92; Part-DB URL (none) -> http://partdb.durbakyta.casa/en/part/92/info; Stock (none) -> 4; Storage Location (none) -> Main Parts Bin; digikey# (none) -> 160-1011-ND; manf (none) -> Lite-On Inc.; manf# (none) -> LTP-3786E
Connections:
- net GND: no longer R8.2
- net at U15.23 (IREF): no longer R8.1
