File: hardware/navbrick.kicad_pcb (KiCad board)
At the start: 2 copper layers, 110.7 x 52.3 mm, 105 parts, among them J50 Conn_01x06_Pin, J51 Conn_01x06_Pin, J52 USB4105-GF-A, J53 Conn_01x02_Pin, J54 Conn_01x02_Pin, J55 Conn_01x03_Pin, J56 Conn_01x03_Pin, J57 Conn_01x08_Pin, J58 Conn_01x08_Pin, Q1 DMP2004VK, Q2 DMP2004VK, Q3 DMP2004VK, Q4 DMP2004VK, SW50 PTS645SK50SMTR92, SW51 PTS645SK50SMTR92, U10 TLC59284, U11 TLC59284, U12 TLC59284, U13 TLC59284, U14 TLC59284, U15 TLC59284, U16 TLC59284, U2 MLX90393SLW-ABA-011, U3 MM74HCT540MTCX, U4 MS5611-01BA, U5 MM74HCT541MTCX, U50 CY7C65223D, U51 SAM-M10Q, U52 LTR-329ALS-01, U53 P3786E, U54 P3786E, U55 P3786E, U56 P3786E, U6 AVR32DA32x-xRXB, U7 FM25L16B, U8 LP2981A-33DBV, U9 TLC59284

Commit message: Initial firmware
Parts:
- Q1, Q2, Q3, Q4: footprint Package_TO_SOT_SMD:SOT-563 -> 0-footprints:SOT-563
- U6: value AVR32DA32x-xRXB -> AVR128DA32x-xRXB
Routing:
- net /Display/PWM6: track 37.5 -> 38.0 mm
