File: hardware/navbrick.kicad_pcb (KiCad board)
At the start: 2 copper layers, 110.7 x 52.3 mm, 105 parts, among them J50 Conn_01x06_Pin, J51 Conn_01x06_Pin, J52 USB4105-GF-A, J53 Conn_01x02_Pin, J54 Conn_01x02_Pin, J55 Conn_01x03_Pin, J56 Conn_01x03_Pin, J57 Conn_01x08_Pin, J58 Conn_01x08_Pin, Q1 DMP2004VK, Q2 DMP2004VK, Q3 DMP2004VK, Q4 DMP2004VK, SW50 PTS645SK50SMTR92, SW51 PTS645SK50SMTR92, U10 TLC59284, U11 TLC59284, U12 TLC59284, U13 TLC59284, U14 TLC59284, U15 TLC59284, U16 TLC59284, U2 MLX90393SLW-ABA-011, U3 MM74HCT540MTCX, U4 MS5611-01BA, U5 MM74HCT541MTCX, U50 CY7C65223D, U51 SAM-M10Q, U52 LTR-329ALS-01, U53 P3786E, U54 P3786E, U55 P3786E, U56 P3786E, U6 AVR128DA32x-xRXB, U7 FM25L16B, U8 LP2981A-33DBV, U9 TLC59284

Commit message: Rev B hardware update
Parts:
- removed JP1, JP2, JP3, JP4, JP5, JP6, JP7, JP8: SolderJumper_3_Open, Jumper:SolderJumper-3_P1.3mm_Open_Pad1.0x1.5mm
- removed JP9: SolderJumper_2_Open, Jumper:SolderJumper-2_P1.3mm_Open_Pad1.0x1.5mm
- removed TP2, TP3, TP4: TestPoint, TestPoint:TestPoint_Pad_D2.0mm
- moved C55 8.02 mm to (-2.29, -37.0), turned to 0 degrees
- moved TP50 7.53 mm to (0.00, -40.9)
- moved C7 6.05 mm to (-41.0, -34.4), turned to -90 degrees
- moved U52 5.16 mm to (-2.29, -39.0), turned to 0 degrees
- moved C14 3.30 mm to (-46.9, -35.4)
- moved C8 3.07 mm to (-39.2, -33.5)
- moved TP51 2.50 mm to (-6.22, -40.9)
- moved U8 1.18 mm to (-44.1, -35.5)
- moved R50 0.74 mm to (-47.4, -41.1)
Connections:
- J52 pad A6: Net-(U50-USBDM) -> Net-(U50-USBDP)
- J52 pad A7: Net-(U50-USBDP) -> Net-(U50-USBDM)
- J52 pad B6: Net-(U50-USBDM) -> Net-(U50-USBDP)
- J52 pad B7: Net-(U50-USBDP) -> Net-(U50-USBDM)
- U3 pad 2: Net-(JP6-C) -> /Display/PWM7
- U3 pad 3: Net-(JP5-C) -> /Display/PWM5
- U3 pad 4: Net-(JP8-C) -> /Display/PWM3
- U3 pad 5: Net-(JP7-C) -> /Display/PWM1
- U3 pad 6: Net-(JP3-C) -> /Display/PWM6
- U3 pad 7: Net-(JP1-C) -> /Display/PWM4
- U3 pad 8: Net-(JP2-C) -> /Display/PWM2
- U3 pad 9: Net-(JP4-C) -> /Display/PWM0
- U51 pad 18: /GPS/RST_N -> unconnected-(U51-~{RESET}-Pad18)
- U6 pad 23: /GPS/RST_N -> unconnected-(U6-PF3-Pad23)
- U6 pad 27: Net-(JP9-B) -> /USB/RxD_1
- U8 pad 4: +3V3 -> unconnected-(U8-NC-Pad4)
- U8 pad 5: unconnected-(U8-NC-Pad5) -> +3V3
Routing:
- net /GPS/RST_N: track 18.1 -> 0.00 mm, vias 1 -> 0
- net /Display/PWM0: track 38.0 -> 24.8 mm
- net Net-(JP4-C): track 12.4 -> 0.00 mm
- net /USB/RxD_1: track 38.5 -> 49.9 mm
- net /Display/PWM2: track 35.3 -> 24.7 mm
- net Net-(JP9-B): track 10.3 -> 0.00 mm
- net Net-(JP7-C): track 10.0 -> 0.00 mm
- net Net-(JP3-C): track 9.77 -> 0.00 mm
- net Net-(JP1-C): track 9.09 -> 0.00 mm, vias 2 -> 0
- net Net-(JP2-C): track 8.64 -> 0.00 mm, vias 2 -> 0
- net /Display/PWM4: track 32.5 -> 24.6 mm
- net Net-(JP5-A): track 7.62 -> 0.00 mm
- net Net-(JP1-B): track 7.62 -> 0.00 mm
- net Net-(JP6-C): track 7.15 -> 0.00 mm
- net /Display/PWM7: track 21.8 -> 28.3 mm
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Other:
- board text added: "NavBrick Alex Mykyta 2023 Rev B"
- board text added: "Rev B"
- board text removed: "NavBrick Alex Mykyta 2023"

Commit message: Add pdf
Parts:
- moved C50 74.4 mm to (9.38, 13.8)
- moved H56 74.4 mm to (15.7, 21.1)
- moved R50 74.4 mm to (7.96, 8.64)
- moved R51 74.4 mm to (7.96, 13.7)
- moved U10 74.4 mm to (86.8, 39.1)
- moved C10 74.4 mm to (13.5, 8.61)
- moved C11 74.4 mm to (2.62, 8.86)
- moved C12 74.4 mm to (5.59, 11.2)
- moved C13 74.4 mm to (3.82, 11.2)
- moved C14 74.4 mm to (8.43, 14.3)
- moved C15 74.4 mm to (59.1, 18.7)
- moved C16 74.4 mm to (105.9, 36.1)
- moved C17 74.4 mm to (93.2, 36.1)
- moved C18 74.4 mm to (80.5, 36.1)
- moved C19 74.4 mm to (67.8, 36.1)
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