File: hardware/GPS.kicad_sch (KiCad schematic)
At the start: 4 parts, among them U16 SAM-M10Q

Commit message: Rev B hardware update
Connections:
- net RST_N: no longer names the net of U16.18 (~{RESET})
- no-connect marks 2 -> 3
Changed lines of the file:
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@@
   (junction (at 121.92 63.5) (diameter 0) (color 0 0 0 0)
   )
+  (no_connect (at 109.22 82.55))
   (no_connect (at 109.22 80.01))
   (no_connect (at 109.22 77.47))
@@
   )
   (wire (pts (xy 124.46 63.5) (xy 121.92 63.5))
-    (stroke (width 0) (type default))
-  )
-  (wire (pts (xy 96.52 82.55) (xy 109.22 82.55))
     (stroke (width 0) (type default))
   )
@@
     (effects (font (size 1.27 1.27)) (justify left))
   )
-  (hierarchical_label "RST_N" (shape input) (at 96.52 82.55 180) (fields_autoplaced)
-    (effects (font (size 1.27 1.27)) (justify right))
-  )
   (symbol (lib_id "0-ic-digital:SAM-M10Q") (at 121.92 77.47 0) (unit 1)
