File: hardware/GPS.kicad_sch (KiCad schematic)
At the start: 4 parts, among them U16 SAM-M10Q

Commit message: Convert to PartDB
Parts:
- C8: symbol 0-passives:C-ceramic -> PartDB:C-Cer-0.1uF-25v-0603; Category (none) -> Capacitors/Ceramic; Manufacturer (none) -> Generic; Part-DB Footprint (none) -> 0603; Part-DB ID (none) -> 4; Part-DB URL (none) -> http://partdb.durbakyta.casa/en/part/4/info; Stock (none) -> 49; Storage Location (none) -> Main Parts Bin; manf (none) -> Generic
- R53, R54: symbol 0-passives:R -> PartDB:R-2.2k-0.1W-0402; Category (none) -> Resistors; DigiKey SPN (none) -> P2.20KLCT-ND; Part-DB Footprint (none) -> 0402; Part-DB ID (none) -> 104; Part-DB URL (none) -> http://partdb.durbakyta.casa/en/part/104/info; Stock (none) -> 0; digikey# (none) -> P2.20KLCT-ND
- U51: renamed from U16; value SAM-M10Q -> SAM-M10Q-00B; symbol 0-ic-digital:SAM-M10Q -> PartDB:SAM-M10Q-00B; Category (none) -> Sensors; DigiKey SPN (none) -> 672-SAM-M10Q-00BCT-ND; MPN (none) -> SAM-M10Q-00B; Manufacturer (none) -> u-blox; Manufacturing Status (none) -> Active; Part-DB ID (none) -> 71; Part-DB URL (none) -> http://partdb.durbakyta.casa/en/part/71/info; Stock (none) -> 1; Storage Location (none) -> Main Parts Bin; digikey# (none) -> 672-SAM-M10Q-00BCT-ND; manf (none) -> u-blox; manf# (none) -> SAM-M10Q-00B
