File: hardware/display.kicad_sch (KiCad schematic)
At the start: 18 parts, among them J2 Conn_01x08_Pin, J3 Conn_01x08_Pin, J4 Conn_01x03_Pin, J5 Conn_01x02_Pin, U14 MM74HCT540MTCX, U4 MM74HCT541MTCX

Commit message: Rev B hardware update
Parts:
- removed JP1, JP2, JP3, JP4, JP5, JP6, JP7, JP8: SolderJumper_3_Open, Jumper:SolderJumper-3_P1.3mm_Open_Pad1.0x1.5mm, symbol 0-passives:SolderJumper_3
Connections:
- net PWM0: now also U14.9 (A7)
- net PWM1: now also U14.5 (A3)
- net PWM2: now also U14.8 (A6)
- net PWM3: now also U14.4 (A2)
- net PWM4: now also U14.7 (A5)
- net PWM5: now also U14.3 (A1)
- net PWM6: now also U14.6 (A4)
- net PWM7: now also U14.2 (A0)
