File: hardware/navbrick.kicad_sch (KiCad schematic)
At the start: 24 parts, among them J50 Conn_01x06_Pin, J51 Conn_01x06_Pin, SW50 PTS645SK50SMTR92, SW51 PTS645SK50SMTR92, U6 AVR128DA32x-xRXB, U7 FM25L16B

Commit message: Convert to PartDB
Parts:
- C5, C53, C54: renamed from C20; symbol 0-passives:C-ceramic -> PartDB:C-Cer-0.1uF-25v-0603; Category (none) -> Capacitors/Ceramic; Manufacturer (none) -> Generic; Part-DB Footprint (none) -> 0603; Part-DB ID (none) -> 4; Part-DB URL (none) -> http://partdb.durbakyta.casa/en/part/4/info; Stock (none) -> 49; Storage Location (none) -> Main Parts Bin; manf (none) -> Generic
- C51, C52: renamed from C20; symbol 0-passives:C-ceramic -> PartDB:C-Cer-0.01uF-50v-0603; Category (none) -> Capacitors/Ceramic; Manufacturer (none) -> Generic; Part-DB Footprint (none) -> 0603; Part-DB ID (none) -> 6; Part-DB URL (none) -> http://partdb.durbakyta.casa/en/part/6/info; Stock (none) -> 69; Storage Location (none) -> Main Parts Bin; manf (none) -> Generic
- R52: symbol 0-passives:R -> PartDB:R-1k-0.1W-0402; Category (none) -> Resistors; DigiKey SPN (none) -> P1.00KLCT-ND; Part-DB Footprint (none) -> 0402; Part-DB ID (none) -> 105; Part-DB URL (none) -> http://partdb.durbakyta.casa/en/part/105/info; Stock (none) -> 0; digikey# (none) -> P1.00KLCT-ND
- SW50, SW51: value PTS645SK50SMTR92 -> PTS645SK50SMTR92 LFS; symbol Switch:SW_Push -> PartDB:PTS645SK50SMTR92 LFS; Category (none) -> Switches; DigiKey SPN (none) -> CKN9087CT-ND; MPN (none) -> PTS645SK50SMTR92 LFS; Manufacturer (none) -> C&K; Manufacturing Status (none) -> Active; Part-DB ID (none) -> 90; Part-DB URL (none) -> http://partdb.durbakyta.casa/en/part/90/info; Stock (none) -> 11; Storage Location (none) -> Main Parts Bin; digikey# (none) -> CKN9087CT-ND; manf (none) -> C&K; manf# (none) -> PTS645SK50SMTR92 LFS
- U6: value AVR128DA32x-xRXB -> AVR128DA32T-I/RXB; symbol 0-Atmel:AVR128DA32x-xRXB -> PartDB:AVR128DA32T-I/RXB; Category (none) -> IC/MCU; DigiKey SPN (none) -> 150-AVR128DA32T-I/RXBCT-ND; MPN (none) -> AVR128DA32T-I/RXB; Manufacturer (none) -> Microchip Technology; Manufacturing Status (none) -> Active; Part-DB ID (none) -> 80; Part-DB URL (none) -> http://partdb.durbakyta.casa/en/part/80/info; Stock (none) -> 1; Storage Location (none) -> Main Parts Bin; digikey# (none) -> 150-AVR128DA32T-I/RXBCT-ND; manf (none) -> Microchip Technology; manf# (none) -> AVR128DA32T-I/RXB
- U7: value FM25L16B -> FM25L16B-GTR; symbol 0-ic-digital:FM25L16B -> PartDB:FM25L16B-GTR; Category (none) -> IC/Memory; DigiKey SPN (none) -> 448-FM25L16B-GTRCT-ND; MPN (none) -> FM25L16B-GTR; Manufacturer (none) -> Infineon Technologies; Manufacturing Status (none) -> Active; Part-DB ID (none) -> 83; Part-DB URL (none) -> http://partdb.durbakyta.casa/en/part/83/info; Stock (none) -> 1; Storage Location (none) -> Main Parts Bin; digikey# (none) -> 448-FM25L16B-GTRCT-ND; manf (none) -> Infineon Technologies; manf# (none) -> FM25L16B-GTR

Commit message: minor fixups
Changed lines of the file:
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@@
 		)
 		(property "Value" "FM25L16B-GTR"
-			(at 229.87 92.71 0)
+			(at 227.076 92.71 0)
 			(show_name no)
 			(do_not_autoplace no)
