File: hardware/sensors.kicad_sch (KiCad schematic)
At the start: 9 parts, among them U15 MLX90393SLW-ABA-011, U17 MS5611-01BA, U52 LTR-329ALS-01

Commit message: Convert to PartDB
Parts:
- C2, C3, C6: symbol 0-passives:C-ceramic -> PartDB:C-Cer-0.1uF-25v-0603; Category (none) -> Capacitors/Ceramic; Manufacturer (none) -> Generic; Part-DB Footprint (none) -> 0603; Part-DB ID (none) -> 4; Part-DB URL (none) -> http://partdb.durbakyta.casa/en/part/4/info; Stock (none) -> 49; Storage Location (none) -> Main Parts Bin; manf (none) -> Generic
- C55: symbol 0-passives:C-ceramic -> PartDB:C-Cer-1uF-10v-0603; Category (none) -> Capacitors/Ceramic; Manufacturer (none) -> Generic; Part-DB Footprint (none) -> 0603; Part-DB ID (none) -> 5; Part-DB URL (none) -> http://partdb.durbakyta.casa/en/part/5/info; Stock (none) -> 63; Storage Location (none) -> Main Parts Bin; manf (none) -> Generic
- U2: renamed from U15; value MLX90393SLW-ABA-011 -> MLX90393SLW-ABA-011-RE; symbol 0-ic-digital:MLX90393SLW -> PartDB:MLX90393SLW-ABA-011-RE; Category (none) -> Sensors; DigiKey SPN (none) -> MLX90393SLW-ABA-011-RECT-ND; MPN (none) -> MLX90393SLW-ABA-011-RE; Manufacturer (none) -> Melexis Technologies NV; Manufacturing Status (none) -> Active; Part-DB ID (none) -> 72; Part-DB URL (none) -> http://partdb.durbakyta.casa/en/part/72/info; Stock (none) -> 1; Storage Location (none) -> Main Parts Bin; digikey# (none) -> MLX90393SLW-ABA-011-RECT-ND; manf (none) -> Melexis Technologies NV; manf# (none) -> MLX90393SLW-ABA-011-RE
- U4: renamed from U17; value MS5611-01BA -> MS561101BA03-50; symbol Sensor_Pressure:MS5611-01BA -> PartDB:MS561101BA03-50; Category (none) -> Sensors; DigiKey SPN (none) -> 223-1622-1-ND; MPN (none) -> MS561101BA03-50; Manufacturer (none) -> TE Connectivity Measurement Specialties; Manufacturing Status (none) -> Active; Part-DB ID (none) -> 70; Part-DB URL (none) -> http://partdb.durbakyta.casa/en/part/70/info; Stock (none) -> 1; Storage Location (none) -> Main Parts Bin; digikey# (none) -> 223-1622-1-ND; manf (none) -> TE Connectivity Measurement Specialties; manf# (none) -> MS561101BA03-50
- U52: footprint 0-footprints:LTR-329ALS-01 -> am-Sensors:LTR-329ALS-01; symbol 0-optoelectronics:LTR-329ALS-01 -> PartDB:LTR-329ALS-01; Category (none) -> Sensors; DigiKey SPN (none) -> 160-2160-1-ND; MPN (none) -> LTR-329ALS-01; Manufacturer (none) -> Lite-On Inc.; Manufacturing Status (none) -> Active; Part-DB ID (none) -> 73; Part-DB URL (none) -> http://partdb.durbakyta.casa/en/part/73/info; Stock (none) -> 1; Storage Location (none) -> Main Parts Bin; digikey# (none) -> 160-2160-1-ND; manf (none) -> Lite-On Inc.; manf# (none) -> LTR-329ALS-01
